Commit message: move head with arrow keys

File: urdf/humanSubject06_48dof.urdf (robot description, URDF)
Before this commit: robot XSensStyleModel_template, 51 links, 50 joints
Joints:
- joint jC1Head_rotx: limit lower=0 upper=1.57 effort=30 velocity=1.0 -> lower=-1.57 upper=1.57 effort=30 velocity=1.0
- joint jC1Head_roty: limit lower=0 upper=1.57 effort=30 velocity=1.0 -> lower=-1.57 upper=1.57 effort=30 velocity=1.0
